Commit message: refactor!: name the package and its files litearm_description
`litearm_description` is the name the consuming stacks use: the CMake guard in
litearm_vr_moveit_config looks up `<package>/urdf/<package>.urdf` through the
ament index and accepts only that name. This package was still called
`litearm`, which is also the name of the superseded arm generation it replaced
in #9, so the same string meant two different arms.

Names only; the model is untouched. The URDF and the nine meshes are
byte-identical to what #9 brought in (joints `joint1..joint7`, links
`joint1..joint7` + `ee_link`, 2.7911 kg, 0 of 7 joint origins shared with the
superseded export). The URDF differs from #9 in 38 of 505 lines and every one
of them is a name.

- SE/litearm/ -> SE/litearm_description/
- urdf/litearm.urdf -> urdf/litearm_description.urdf
- config/joint_names_litearm.yaml -> config/joint_names_litearm_description.yaml
- package.xml: `<name>` and the package reference in `<description>`
- CMakeLists.txt: `project()`
- URDF: `<robot name>` and the nine `package://` mesh URIs
- both launch files: the share directory, the URDF path and the Gazebo entity
- README.md and README.zh-CN.md, at the repository root and in the package

Not renamed: rviz/display.rviz, whose name carries no package name, and the
provenance notes that point at the `litearm` package inside litearm-stm32.

Verified: xmllint accepts package.xml and the URDF, `check_urdf` parses the
tree (base_link -> joint1..joint7 -> ee_link), both launch files compile, every
`package://` mesh resolves case-sensitively, every link and joint name is
lowercase, and the CI mesh check finds no unknown package.

BREAKING CHANGE: anything that refers to the package as `litearm`, to
`urdf/litearm.urdf` or to `package://litearm/...` must switch to
`litearm_description`.

File: SE/litearm_description/urdf/litearm_description.urdf (robot description, URDF)
Before this commit: robot litearm, 9 links, 8 joints
Links:
- link base_link: geometry collision mesh filename=package://litearm_description/meshes/base_link.STL; visual mesh filename=package://litearm_description/meshes/base_link.STL
- link ee_link: geometry collision mesh filename=package://litearm_description/meshes/ee_link.STL; visual mesh filename=package://litearm_description/meshes/ee_link.STL
- link joint1: geometry collision mesh filename=package://litearm_description/meshes/joint1.STL; visual mesh filename=package://litearm_description/meshes/joint1.STL
- link joint2: geometry collision mesh filename=package://litearm_description/meshes/joint2.STL; visual mesh filename=package://litearm_description/meshes/joint2.STL
- link joint3: geometry collision mesh filename=package://litearm_description/meshes/joint3.STL; visual mesh filename=package://litearm_description/meshes/joint3.STL
- link joint4: geometry collision mesh filename=package://litearm_description/meshes/joint4.STL; visual mesh filename=package://litearm_description/meshes/joint4.STL
- link joint5: geometry collision mesh filename=package://litearm_description/meshes/joint5.STL; visual mesh filename=package://litearm_description/meshes/joint5.STL
- link joint6: geometry collision mesh filename=package://litearm_description/meshes/joint6.STL; visual mesh filename=package://litearm_description/meshes/joint6.STL
- link joint7: geometry collision mesh filename=package://litearm_description/meshes/joint7.STL; visual mesh filename=package://litearm_description/meshes/joint7.STL
